File: Intercom.kicad_sch (KiCad schematic)
At the start: 17 parts, among them J1 To other, P1 22k, SW1 SW_Push, U1 LM386

Commit message: Rename to Intercom
Other:
- title: Gegensprechanlage -> Intercom
Changed lines of the file:
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@@
   (paper "A4")
   (title_block
-    (title "Gegensprechanlage")
+    (title "Intercom")
     (date "2022-12-08")
     (rev "1.0")
