File: Intercom.kicad_pcb (KiCad board)
At the start: 2 copper layers, 51.5 x 28.6 mm, 17 parts, among them P1 22k, SW1 SW_Push, U1 LM386

Commit message: Update drill file
Other:
- board text added: "Intercom V1.0 9.12.22"
- board text removed: "V1.0 - 9.12.22"
Changed lines of the file:
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@@
     (fp_line (start 6.7 13.95) (end 6.7 -3.95) (layer "F.Fab") (width 0.1))
     (fp_line (start -18.8 8) (end -8.8 8) (layer "F.Fab") (width 0.1))
-    (pad "1" thru_hole oval (at 0 0 180) (size 4.5 3) (drill 0.8) (layers *.Cu *.Mask)
+    (pad "1" thru_hole oval (at 0 0 180) (size 4.5 3) (drill 0.7) (layers *.Cu *.Mask)
       (net 10 "Net-(C2-Pad1)") (pinfunction "1") (pintype "passive"))
     (pad "2" thru_hole oval (at 0 5 180) (size 4.5 3) (drill 0.8) (layers *.Cu *.Mask)
@@
     (effects (font (size 1 1) (thickness 0.15)))
   )
-  (gr_text "V1.0 - 9.12.22" (at 121.5136 91.4654 90) (layer "F.SilkS")
+  (gr_text "Intercom V1.0\n9.12.22" (at 120.2182 78.613) (layer "F.SilkS")
     (effects (font (size 1 1) (thickness 0.15)))
   )
